Commit message: Add files via upload

File: scout_gazebo/urdf/base.xacro (robot description, xacro)
@@ -29,5 +29,6 @@
             <origin xyz="0 0 0" rpy="0 0 0" />
             <geometry>
-                <box size="${base_x_size} ${base_y_size} ${base_z_size}"/>
+                <!--<box size="${base_x_size} ${base_y_size} ${base_z_size}"/>-->
+                <mesh filename="package://scout_gazebo/meshes/base_link.dae" />
             </geometry>
         </visual>

File: scout_gazebo/urdf/scout_wheel_type1.xacro (robot description, xacro)
@@ -32,7 +32,7 @@
             </inertial>
             <visual>
-                <origin xyz="0 0 0" rpy="${M_PI/2} 0 0" />
+                <origin xyz="0 0 0" rpy="0 0 0" />
                 <geometry>
-                    <cylinder length="${wheel_length}" radius="${wheel_radius}" />
+                    <mesh filename="package://scout_gazebo/meshes/wheel_type1.dae" />
                 </geometry>
             </visual>
@@ -50,7 +50,4 @@
             <axis xyz="0 -1 0" rpy="0 0 0" />
         </joint>
-        <gazebo reference="${wheel_prefix}_wheel_link">
-        	<material>Gazebo/Black</material>
-    	</gazebo>
     </xacro:macro>
 </robot>

File: scout_gazebo/urdf/scout_wheel_type2.xacro (robot description, xacro)
@@ -32,7 +32,7 @@
             </inertial>
             <visual>
-                <origin xyz="0 0 0" rpy="${M_PI/2} 0 0" />
+                <origin xyz="0 0 0" rpy="0 0 0" />
                 <geometry>
-                    <cylinder length="${wheel_length}" radius="${wheel_radius}" />
+                    <mesh filename="package://scout_gazebo/meshes/wheel_type2.dae" />
                 </geometry>
             </visual>
@@ -50,7 +50,4 @@
             <axis xyz="0 -1 0" rpy="0 0 0" />
         </joint>
-        <gazebo reference="${wheel_prefix}_wheel_link">
-        	<material>Gazebo/Black</material>
-    	</gazebo>
     </xacro:macro>
 </robot>
